File: electronics/POC_temp_sens/POC_temp_sens.kicad_pcb (KiCad board)
At the start: 2 copper layers, 106.7 x 78.7 mm, 53 parts, among them J1 Conn_01x06, J2 Conn_01x06, J3 Conn_01x05, J4 nuclone_left, J5 nuclone_right, U1 74XX4051, U2 OP07C, U3 LM358, U5 74XX4051

Commit message: added more resistors to multiplexers
Parts:
- added R30: 47K, SquantorResistor:R_0603_hand, B.Cu at (68.6, 39.4)
- added R31: 47K, SquantorResistor:R_0603_hand, B.Cu at (45.7, 39.4)
Connections:
- J5 pad 5: unconnected-(J5-Pin_5-Pad5) -> GND
- J5 pad 6: unconnected-(J5-Pin_6-Pad6) -> GND
- U1 pad 6: GND -> Net-(U1-!E)
- U5 pad 6: GND -> Net-(U5-!E)
Routing:
- net GND: track 91.9 -> 181.6 mm, vias 3 -> 2
- net /+3.3V: track 0.00 -> 55.9 mm, vias 0 -> 1
- net /-5V: track 78.0 -> 132.6 mm, vias 1 -> 3
- net /+8V: track 21.4 -> 44.2 mm, vias 2 -> 3

Commit message: small changes, updated HSI
Parts:
- moved R7 1.80 mm to (57.1, 61.0), turned to 0 degrees
Connections:
- R7 pad 1: GND -> /+8V
Changed lines of the file:
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@@
 	(footprint "SquantorResistor:R_0603_hand"
 		(layer "B.Cu")
-		(at 58.42 59.69 -90)
+		(at 57.15 60.96)
 		(descr "Resistor SMD 0603, reflow soldering, Vishay (see dcrcw.pdf)")
 		(tags "resistor 0603")
 		(property "Reference" "R7"
-			(at 0 1.2 90)
+			(at 0 1.2 360)
 			(layer "B.SilkS")
 			(effects
@@
 		)
 		(property "Value" "82K"
-			(at 0 -1.2 90)
+			(at 0 -1.2 360)
 			(layer "B.Fab")
 			(effects
@@
 		)
 		(property "Footprint" "SquantorResistor:R_0603_hand"
-			(at 0 0 90)
+			(at 0 0 360)
 			(layer "B.Fab")
 			(hide yes)
@@
 		)
 		(property "Datasheet" ""
-			(at 0 0 90)
+			(at 0 0 360)
 			(layer "B.Fab")
 			(hide yes)
@@
 		)
 		(property "Description" "Resistor"
-			(at 0 0 90)
+			(at 0 0 360)
 			(layer "B.Fab")
 			(hide yes)
@@
 		)
 		(fp_line
-			(start 1.4 0.65)
+			(start -1.4 -0.65)
 			(end -1.4 0.65)
 			(stroke
@@
 		)
 		(fp_line
-			(start -1.4 -0.65)
-			(end -1.4 0.65)
+			(start 1.4 -0.65)
+			(end -1.4 -0.65)
 			(stroke
 				(width 0.05)
@@
 		)
 		(fp_line
-			(start 1.4 -0.65)
-			(end -1.4 -0.65)
+			(start 1.4 0.65)
+			(end -1.4 0.65)
 			(stroke
 				(width 0.05)
@@
 		)
 		(fp_line
+			(start -0.8 -0.4)
+			(end 0.8 -0.4)
+			(stroke
+				(width 0.1)
+				(type solid)
+			)
+			(layer "B.Fab")
+		)
+		(fp_line
 			(start -0.8 0.4)
 			(end -0.8 -0.4)
+			(stroke
+				(width 0.1)
+				(type solid)
+			)
+			(layer "B.Fab")
+		)
+		(fp_line
+			(start 0.8 -0.4)
+			(end 0.8 0.4)
 			(stroke
 				(width 0.1)
@@
 			(layer "B.Fab")
 		)
-		(fp_line
-			(start -0.8 -0.4)
-			(end 0.8 -0.4)
-			(stroke
-				(width 0.1)
-				(type solid)
-			)
-			(layer "B.Fab")
-		)
-		(fp_line
-			(start 0.8 -0.4)
-			(end 0.8 0.4)
-			(stroke
-				(width 0.1)
-				(type solid)
-			)
-			(layer "B.Fab")
-		)
 		(pad "1" smd roundrect
-			(at -0.85 0 270)
+			(at -0.85 0)
 			(size 0.7 0.9)
 			(layers "B.Cu" "B.Paste" "B.Mask")
 			(roundrect_rratio 0.1428571429)
-			(net 2 "GND")
+			(net 6 "/+8V")
 			(pintype "passive")
 		)
 		(pad "2" smd roundrect
-			(at 0.85 0 270)
+			(at 0.85 0)
 			(size 0.7 0.9)
 			(layers "B.Cu" "B.Paste" "B.Mask")
