File: electronics/POC_temp_sens/POC_temp_sens.kicad_sch (KiCad schematic)
At the start: 53 parts, among them J1 Conn_01x06, J2 Conn_01x06, J3 Conn_01x05, J4 nuclone_left, J5 nuclone_right, U1 74XX4051, U2 OP07C, U3 LM358, U5 74XX4051

Commit message: added more resistors to multiplexers
Parts:
- added R30, R31: 47K, SquantorResistor:R_0603_hand, symbol Device:R
Connections:
- net GND: now also J5.5 (Pin_5), J5.6 (Pin_6), R30.1, R31.1; no longer U1.6 (!E), U5.6 (!E)
- new net: R30.2, U5.6 (!E)
- new net: R31.2, U1.6 (!E)

Commit message: small changes, updated HSI
Connections:
- net +8V: now also R7.1
- net GND: no longer R7.1
Changed lines of the file:
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@@
+		)
+	)
+	(label "+8V"
+		(at 143.51 50.8 180)
+		(fields_autoplaced yes)
+		(effects
+			(font
+				(size 1.27 1.27)
+			)
+			(justify right bottom)
 		)
 	)
@@
 					(unit 1)
 				)
-			)
-		)
-	)
-	(symbol
-		(lib_id "power:GND")
-		(at 143.51 50.8 270)
-		(unit 1)
-		(exclude_from_sim no)
-		(in_bom yes)
-		(on_board yes)
-		(dnp no)
-		(fields_autoplaced yes)
-		(property "Reference" "#PWR07"
-			(at 137.16 50.8 0)
-			(effects
-				(font
-					(size 1.27 1.27)
-				)
-				(hide yes)
-			)
-		)
-		(property "Value" "GND"
-			(at 139.7 50.7999 90)
-			(effects
-				(font
-					(size 1.27 1.27)
-				)
-				(justify right)
-			)
-		)
-		(property "Footprint" ""
-			(at 143.51 50.8 0)
-			(effects
-				(font
-					(size 1.27 1.27)
-				)
-				(hide yes)
-			)
-		)
-		(property "Datasheet" ""
-			(at 143.51 50.8 0)
-			(effects
-				(font
-					(size 1.27 1.27)
-				)
-				(hide yes)
-			)
-		)
-		(property "Description" "Power symbol creates a global label with name \"GND\" , ground"
-			(at 143.51 50.8 0)
-			(effects
-				(font
-					(size 1.27 1.27)
-				)
-				(hide yes)
-			)
-		)
-		(pin "1"
-		)
-		(instances
-			(project "T245_sense_protoboard"
-				(path "/646d9e91-59b4-4865-a2fc-29780ed32563"
-					(reference "#PWR07")
-					(unit 1)
-				)
