File: electronics/module_dual_powerstage/module_dual_powerstage.kicad_pcb (KiCad board)
At the start: 2 copper layers, 2 parts

Commit message: Schematic and layout done, review needed
Parts:
- added C1: 1u, SquantorCapacitor:C_0805+0603, F.Cu at (185.3, 50.6)
- added C2: 1u, SquantorCapacitor:C_0805+0603, F.Cu at (168.2, 46.0)
- added C3: 1u, SquantorCapacitor:C_0805+0603, F.Cu at (168.2, 56.2)
- added D1: BAV70, SquantorIC:SOT23-3, F.Cu at (167.3, 52.6)
- added D2: BZT52C18, SquantorDiodes:SOD-323-nexperia-hand, F.Cu at (166.3, 46.1)
- added D3: BAS316, SquantorDiodes:SOD-323-nexperia-hand, F.Cu at (160.6, 45.3)
- added D4: BAS316, SquantorDiodes:SOD-323-nexperia-hand, F.Cu at (160.6, 55.0)
- added D5: BAV70, SquantorIC:SOT23-3, F.Cu at (167.4, 62.8)
- added D6: BZT52C18, SquantorDiodes:SOD-323-nexperia-hand, F.Cu at (166.3, 56.1)
- added J1: Conn_01x04, SquantorConnectors:Header-0254-1X04-H010, F.Cu at (154.9, 54.6)
- added J2: Conn_01x04, SquantorConnectors:Header-0254-1X04-H010, F.Cu at (188.0, 53.3)
- added OP1: TLP521-4, SquantorIC:DIP-16_W7.62mm, F.Cu at (174.0, 54.6)
- added Q1: 60V4A, SquantorIC:SOIC-8, F.Cu at (161.5, 49.4)
- added Q2: BC858B, SquantorIC:SOT23-3, F.Cu at (180.7, 46.7)
- added Q3: BC847A, SquantorIC:SOT23-3, F.Cu at (180.7, 52.9)
- added Q4: BC858B, SquantorIC:SOT23-3, F.Cu at (180.7, 56.3)
- added Q5: BC847A, SquantorIC:SOT23-3, F.Cu at (180.7, 62.4)
- added Q6: 60V4A, SquantorIC:SOIC-8, F.Cu at (161.5, 59.5)
- added R1: 10M, SquantorResistor:R_0603_hand, F.Cu at (161.0, 53.4)
- added R10: 10K, SquantorResistor:R_0603_hand, F.Cu at (183.2, 52.7)
- added R11: 10K, SquantorResistor:R_0603_hand, F.Cu at (184.5, 46.7)
- added R12: 330, SquantorResistor:R_0603_hand, F.Cu at (180.4, 58.7)
- added R13: 330, SquantorResistor:R_0603_hand, F.Cu at (180.4, 60.0)
- added R14: 6K8, SquantorResistor:R_0603_hand, F.Cu at (183.2, 56.3)
- added R15: 10K, SquantorResistor:R_0603_hand, F.Cu at (183.2, 59.3)
- added R16: 10K, SquantorResistor:R_0603_hand, F.Cu at (183.2, 62.3)
- added R17: 10K, SquantorResistor:R_0603_hand, F.Cu at (184.5, 59.3)
- added R18: 10M, SquantorResistor:R_0603_hand, F.Cu at (161.0, 63.5)
- added R19: 5K6, SquantorResistor:R_0603_hand, F.Cu at (167.1, 59.5)
- added R2: 5K6, SquantorResistor:R_0603_hand, F.Cu at (167.1, 49.3)
- added R20: 1M, SquantorResistor:R_0603_hand, F.Cu at (164.0, 63.5)
- added R21: 1K5, SquantorResistor:R_0603_hand, F.Cu at (168.4, 59.5)
- added R22: 2K2, SquantorResistor:R_0603_hand, F.Cu at (163.8, 55.2)
- added R3: 1M, SquantorResistor:R_0603_hand, F.Cu at (164.0, 53.4)
- added R4: 1K5, SquantorResistor:R_0603_hand, F.Cu at (168.4, 49.3)
- added R5: 2K2, SquantorResistor:R_0603_hand, F.Cu at (163.8, 44.9)
- added R6: 330, SquantorResistor:R_0603_hand, F.Cu at (180.4, 49.1)
- added R7: 330, SquantorResistor:R_0603_hand, F.Cu at (180.4, 50.5)
- added R8: 6K8, SquantorResistor:R_0603_hand, F.Cu at (183.2, 46.7)
- added R9: 10K, SquantorResistor:R_0603_hand, F.Cu at (183.2, 49.7)
- N1: renamed from N2; moved to B.Cu
- N2: renamed from N1; value 20231214 -> 20250926; moved to B.Cu
- moved N1 50.3 mm to (174.0, 51.8), turned to 180 degrees
- moved N2 50.3 mm to (174.0, 55.5), turned to 180 degrees
Routing:
- net /V3.3: track 0.00 -> 35.6 mm, vias 0 -> 4
- net /dual_nmos_switch/SW_S2: track 0.00 -> 23.9 mm
- net /dual_nmos_switch/SW_S1: track 0.00 -> 23.8 mm, vias 0 -> 1
- net /AC1_IN: track 0.00 -> 14.6 mm, vias 0 -> 5
- net /dual_nmos_switch/SW_G2: track 0.00 -> 12.4 mm
- net /dual_nmos_switch/SW_G1: track 0.00 -> 12.1 mm
- net /SW1: track 0.00 -> 11.7 mm
- net /GND: track 0.00 -> 9.28 mm, vias 0 -> 5
- net /SW2: track 0.00 -> 8.28 mm
- net /AC2_IN: track 0.00 -> 7.87 mm, vias 0 -> 5
- net Net-(D1-K2): track 0.00 -> 6.85 mm
- net Net-(D5-K2): track 0.00 -> 6.73 mm
- net Net-(D6-K): track 0.00 -> 5.89 mm
- net Net-(D2-K): track 0.00 -> 5.82 mm
- net /AC2_OUT: track 0.00 -> 5.27 mm, vias 0 -> 5
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- added copper zone on B.Cu, net /AC1_IN
- added copper zone on F.Cu, net /AC1_IN
- added copper zone on B.Cu, net /AC1_OUT
- added copper zone on F.Cu, net /AC1_OUT
- added copper zone on B.Cu, net /AC2_IN
- added copper zone on F.Cu, net /AC2_IN
- added copper zone on B.Cu, net /AC2_OUT
- added copper zone on F.Cu, net /AC2_OUT
- added copper zone on B.Cu, net /GND
- added copper zone on F.Cu, net /GND
Other:
- board outline added: 36.3 x 21.4 mm
